File: hardware/4x_laser_controller/4x_laser_controller.kicad_pcb (KiCad board)
At the start: 4 copper layers, 70.8 x 100 mm, 141 parts, among them J1 ILDA4, J2 Conn_02x05_Odd_Even, J3 ILDA3, J4 ILDA1, J5 ILDA2, J6 Conn_02x05_Odd_Even, J7 AUDIO_IN, J8 Conn_01x03, J9 MODE, SW1 INTERLOCK4, SW2 INTERLOCK3, SW3 INTERLOCK1, SW4 INTERLOCK2, U1 L7805, U10 Teensy4.1, U2 TL074, U3 74LS125, U4 TL074, U5 74LS125, U6 TL074, U7 TL074, U8 74LS125, U9 DAC7578xPW

Commit message: Added calibration routines and changed longs to ints and floats
Parts:
- removed the R45 at (130.7, 89.1)
- removed the R48 at (132.2, 89.1)
- removed the R62 at (124.8, 82.7)
- removed the U9 at (128.4, 82.8)
- added C14: 0.1u, Capacitor_SMD:C_0603_1608Metric, F.Cu at (124.3, 89.9)
- added C19: 0.1u, Capacitor_SMD:C_0603_1608Metric, F.Cu at (124.4, 80.0)
- added C8: 0.1u, Capacitor_SMD:C_0603_1608Metric, F.Cu at (145.5, 89.6)
- added U10: MCP4922-EST, Package_SO:TSSOP-14_4.4x5mm_P0.65mm, F.Cu at (128.0, 88.0)
- added U11: MCP4922-EST, Package_SO:TSSOP-14_4.4x5mm_P0.65mm, F.Cu at (128.0, 78.0)
- added U12: MCP4922-EST, Package_SO:TSSOP-14_4.4x5mm_P0.65mm, F.Cu at (108.8, 88.2)
- added U7: MCP4922-EST, Package_SO:TSSOP-14_4.4x5mm_P0.65mm, F.Cu at (149.1, 87.7)
- moved C6 29.1 mm to (105.2, 90.2)
- moved R53 21.9 mm to (105.2, 85.9)
- moved R8 20.6 mm to (148.9, 83.0), turned to 180 degrees
- moved R9 18.4 mm to (145.5, 85.6)
- moved R52 17.2 mm to (108.5, 83.4), turned to 180 degrees
- moved R38 15.9 mm to (127.5, 73.3), turned to 180 degrees
- moved R24 10.5 mm to (124.3, 86.4)
- moved R23 5.81 mm to (127.4, 83.3), turned to 180 degrees
- moved R39 2.16 mm to (124.4, 76.1)
- renumbered C8 to C10, C9 to C11, C11 to C12, C12 to C13, C13 to C15, C14 to C16, C15 to C17, C16 to C18, C17 to C20, C18 to C21, C10 to C6, C6 to C7, C7 to C9, R46 to R45, R47 to R46, R49 to R47, R50 to R48, R51 to R49, R52 to R50, R53 to R51, R54 to R52, R55 to R53, R56 to R54, R57 to R55, R58 to R56, R59 to R57, R60 to R58, R61 to R59, R63 to R60, R64 to R61, R65 to R62, R66 to R63, R67 to R64, R68 to R65, R69 to R66, R70 to R67, R71 to R68, R72 to R69, R73 to R70, R74 to R71, R75 to R72, R76 to R73, R77 to R74, R78 to R75, R79 to R76, R80 to R77, R81 to R78, R82 to R79, R83 to R80, R84 to R81, R85 to R82, R86 to R83, R87 to R84, R88 to R85, R89 to R86, R90 to R87, R91 to R88, U10 to U13, U7 to U8, U8 to U9
Connections:
- U13 pad 13: B_LO4 -> MOSI
- U13 pad 14: unconnected-(U10-Pad14) -> MISO
- U13 pad 24: unconnected-(U10-Pad24) -> B_LO4
- U13 pad 28: unconnected-(U10-Pad28) -> CS4
- U13 pad 29: unconnected-(U10-Pad29) -> CS3
- U13 pad 30: unconnected-(U10-Pad30) -> CS2
- U13 pad 31: unconnected-(U10-Pad31) -> CS1
- U13 pad 35: unconnected-(U10-Pad35) -> SCK
Routing:
- net SCK: track 0.00 -> 108.8 mm, vias 0 -> 4
- net +3V3: track 116.5 -> 189.8 mm, vias 3 -> 6
- net MOSI: track 0.00 -> 68.9 mm, vias 0 -> 4
- net SCL: track 44.2 -> 0.00 mm, vias 1 -> 0
- net CS1: track 0.00 -> 44.0 mm
- net SDA: track 40.7 -> 0.00 mm, vias 1 -> 0
- net CS3: track 0.00 -> 37.7 mm
- net Net-(R13-Pad1): track 72.7 -> 43.2 mm
- net CS2: track 0.00 -> 25.5 mm
- net CS4: track 0.00 -> 23.4 mm, vias 0 -> 1
- net Net-(R52-Pad2): track 62.4 -> 42.8 mm
- net Net-(R38-Pad2): track 51.7 -> 33.4 mm
- net B_LO4: track 31.4 -> 46.0 mm
- net Net-(R24-Pad2): track 33.2 -> 43.8 mm
- net Net-(R23-Pad2): track 60.7 -> 50.3 mm
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Other:
- board text added: "4x Laser Controller Rev 3 Alex DeBoni"
- board text removed: "4x Laser Controller Rev 2 Alex DeBoni"
