File: hardware/4x_laser_controller/4x_laser_controller.kicad_sch (KiCad schematic)
At the start: 141 parts, among them J1 ILDA4, J2 Conn_02x05_Odd_Even, J3 ILDA3, J4 ILDA1, J5 ILDA2, J6 Conn_02x05_Odd_Even, J7 AUDIO_IN, J8 Conn_01x03, J9 MODE, SW1 INTERLOCK4, SW2 INTERLOCK3, SW3 INTERLOCK1, SW4 INTERLOCK2, U1 L7805, U10 Teensy4.1, U2 TL074, U3 74LS125, U4 TL074, U5 74LS125, U6 TL074, U7 TL074, U8 74LS125, U9 DAC7578xPW

Commit message: Added calibration routines and changed longs to ints and floats
Parts:
- removed R45, R48, R62: 10k, Resistor_SMD:R_0603_1608Metric, symbol Device:R_US
- removed U9: DAC7578xPW, Package_SO:TSSOP-16_4.4x5mm_P0.65mm, symbol Analog_DAC:DAC7578xPW
- added C14, C19, C8: 0.1u, Capacitor_SMD:C_0603_1608Metric, symbol Device:C
- added U10, U11, U12, U7: MCP4922-EST, Package_SO:TSSOP-14_4.4x5mm_P0.65mm, symbol Analog_DAC:MCP4922-EST
- renumbered C8 to C10, C9 to C11, C11 to C12, C12 to C13, C13 to C15, C14 to C16, C15 to C17, C16 to C18, C17 to C20, C18 to C21, C10 to C6, C6 to C7, C7 to C9, R46 to R45, R47 to R46, R49 to R47, R50 to R48, R51 to R49, R52 to R50, R53 to R51, R54 to R52, R55 to R53, R56 to R54, R57 to R55, R58 to R56, R59 to R57, R60 to R58, R61 to R59, R63 to R60, R64 to R61, R65 to R62, R66 to R63, R67 to R64, R68 to R65, R69 to R66, R70 to R67, R71 to R68, R72 to R69, R73 to R70, R74 to R71, R75 to R72, R76 to R73, R77 to R74, R78 to R75, R79 to R76, R80 to R77, R81 to R78, R82 to R79, R83 to R80, R84 to R81, R85 to R82, R86 to R83, R87 to R84, R88 to R85, R89 to R86, R90 to R87, R91 to R88, U10 to U13, U7 to U8, U8 to U9
Connections:
- net +3V3: now also C14.2, C19.2, C8.2, U10.1 (VDD), U10.11 (VrefB), U10.13 (VrefA), U10.9 (~{SHDN}), U11.1 (VDD), U11.11 (VrefB), U11.13 (VrefA), U11.9 (~{SHDN}), U12.1 (VDD), U12.11 (VrefB), U12.13 (VrefA), U12.9 (~{SHDN}), U7.1 (VDD), U7.11 (VrefB), U7.13 (VrefA), U7.9 (~{SHDN})
- net B_LO4: now also U13.24 (32_OUT1B); no longer U13.13 (11_MOSI_CTX1)
- net GND: now also C14.1, C19.1, C8.1, U10.12 (AVSS), U10.8 (~{LDAC}), U11.12 (AVSS), U11.8 (~{LDAC}), U12.12 (AVSS), U12.8 (~{LDAC}), U7.12 (AVSS), U7.8 (~{LDAC})
- net X1_LO: now also U7.14 (VoutA)
- net X2_LO: now also U10.14 (VoutA)
- net X3_LO: now also U11.14 (VoutA)
- net X4_LO: now also U12.14 (VoutA)
- net Y1_LO: now also U7.10 (VoutB)
- net Y2_LO: now also U10.10 (VoutB)
- net Y3_LO: now also U11.10 (VoutB)
- net Y4_LO: now also U12.10 (VoutB)
- net MISO: now reaches U13.14 (12_MISO_MQSL)
- net CS4: now reaches U13.28 (36_CS)
- net CS4: now also U12.3 (~{CS})
- net CS3: now reaches U13.29 (37_CS)
- net CS3: now also U11.3 (~{CS})
- net CS2: now reaches U13.30 (38_CS1_IN1)
- net CS2: now also U10.3 (~{CS})
- net CS1: now reaches U13.31 (39_MISO1_OUT1A)
- net CS1: now also U7.3 (~{CS})
- net SCK: now reaches U13.35 (13_SCK_LED)
- net SCK: now also U10.4 (SCK), U11.4 (SCK), U12.4 (SCK), U7.4 (SCK)
- new net MOSI: U10.5 (SDI), U11.5 (SDI), U12.5 (SDI), U13.13 (11_MOSI_CTX1), U7.5 (SDI)
Other:
- moved on the sheet: C6, D3, D4, D5, D6, R69, R71, R73, R78, U13
