File: hardware/mega_laser_driver/mega_laser_driver.kicad_pcb (KiCad board)
At the start: 2 copper layers, 100 x 100 mm, 90 parts, among them J1 Conn_01x03, J10 Conn_01x02, J11 Conn_01x02, J2 Conn_01x02, J3 Conn_01x02, J4 Conn_01x02, J5 Conn_01x02, J6 Conn_01x02, J7 Conn_01x02, J8 Conn_02x03_Odd_Even, J9 Conn_01x03, K1 G6S-2, Q1 BD139, Q2 BD139, Q3 BD139, U1 LM2576S-ADJ, U2 LM324, U3 LM324, U4 LM2576S-ADJ, U5 LM2576S-ADJ

Commit message: Added new hardware
Parts:
- removed J1: Conn_01x03, Connector_JST:JST_XH_B3B-XH-A_1x03_P2.50mm_Vertical
- removed J10: Conn_01x02, Connector_JST:JST_XH_B2B-XH-A_1x02_P2.50mm_Vertical
- removed J11: Conn_01x02, Connector_PinHeader_2.54mm:PinHeader_1x02_P2.54mm_Vertical
- removed K1: G6S-2, Relay_THT:Relay_DPDT_Omron_G6S-2
- added C10: 220u, Capacitor_SMD:CP_Elec_6.3x7.7, F.Cu at (43.5, 75.0)
- added C11: 220u, Capacitor_SMD:CP_Elec_6.3x7.7, F.Cu at (43.5, 83.0)
- added C9: 220u, Capacitor_SMD:CP_Elec_6.3x7.7, F.Cu at (71.1, 90.7)
- added D13: LED, LED_SMD:LED_0603_1608Metric, F.Cu at (66.5, 87.5)
- added D14: SS54, Diode_SMD:D_SMA, F.Cu at (71.1, 97.8)
- added D15: LED, LED_SMD:LED_0603_1608Metric, F.Cu at (64.8, 87.5)
- added J12: DB25_Plug_MountingHoles, Connector_Dsub:DSUB-25_Male_Horizontal_P2.77x2.84mm_EdgePinOffset7.70mm_Housed_MountingHolesOffset9.12mm, F.Cu at (19.0, 89.0)
- added K2: G5Q-1A-DC12, Relay_THT:Relay_SPST_Omron-G5Q-1A, F.Cu at (10.5, 79.0)
- added Q4: TIP120, Package_TO_SOT_THT:TO-220-3_Horizontal_TabDown, F.Cu at (17.5, 30.7)
- added R31: 100, Resistor_SMD:R_0603_1608Metric, F.Cu at (8.50, 84.3)
- added R32: 560, Resistor_SMD:R_0603_1608Metric, F.Cu at (66.5, 90.7)
- added R33: 680, Resistor_SMD:R_0603_1608Metric, F.Cu at (64.8, 90.7)
- added SW1: SW_SPDT, Button_Switch_SMD:SW_SPDT_PCM12, F.Cu at (2.50, 85.5)
- added U6: TEN20-2422WIN, AlexCustom:PYBE30-Q24-D15, F.Cu at (74.0, 73.0)
- C12, C13, C3, C4, C5, C6: value 1000u -> 220u; footprint Capacitor_SMD:CP_Elec_10x10 -> Capacitor_SMD:CP_Elec_6.3x7.7
- C15: footprint Capacitor_SMD:CP_Elec_6.3x5.4_Nichicon -> Capacitor_SMD:C_1210_3225Metric
- D1, D2, D9: footprint Diode_SMD:D_SMA_Handsoldering -> Diode_SMD:D_SOD-123
- J2, J3, J4: value Conn_01x02 -> Conn_01x03; footprint Connector_JST:JST_XH_B2B-XH-A_1x02_P2.50mm_Vertical -> Connector_JST:JST_XH_B3B-XH-A_1x03_P2.50mm_Vertical
- J9: value Conn_01x03 -> Barrel_Jack_Switch; footprint Connector_PinHeader_2.54mm:PinHeader_1x03_P2.54mm_Vertical -> Connector_BarrelJack:BarrelJack_CLIFF_FC681465S_SMT_Horizontal
- Q1, Q2: value BD139 -> TIP120; footprint Package_TO_SOT_THT:TO-126-3_Horizontal_TabDown -> Package_TO_SOT_THT:TO-220-3_Horizontal_TabDown
- Q3: value BD139 -> 2N7002; footprint Package_TO_SOT_THT:TO-126-3_Horizontal_TabDown -> Package_TO_SOT_SMD:SOT-23
- moved R3 271.4 mm to (30.0, 41.0)
- moved C12 251.0 mm to (12.5, 40.0), turned to 90 degrees
- moved R11 248.5 mm to (36.0, 15.6), turned to 180 degrees
- moved C4 247.6 mm to (45.5, 40.0), turned to 90 degrees
- moved C6 241.1 mm to (38.0, 40.0), turned to 90 degrees
- moved R12 240.1 mm to (36.0, 17.9), turned to 180 degrees
- moved R14 222.8 mm to (66.0, 15.6), turned to 180 degrees
- moved R15 216.0 mm to (66.0, 17.9), turned to 180 degrees
- moved D2 212.0 mm to (54.0, 54.0)
- moved R4 211.1 mm to (63.0, 41.0)
- moved RV1 205.0 mm to (31.0, 50.0), turned to -90 degrees
- moved C3 200.2 mm to (78.5, 40.0), turned to 90 degrees
- moved RV2 198.1 mm to (64.0, 50.0), turned to -90 degrees
- moved D9 197.8 mm to (87.0, 54.0)
- moved H2 197.8 mm to (4.00, 4.00)
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Connections:
- C14 pad 1: Net-(C14-Pad1) -> X+
- C15 pad 1: Net-(C15-Pad1) -> GND
- C15 pad 2: GND -> Net-(U3D-+)
- D10 pad 1: Net-(D10-Pad1) -> +12V
- D10 pad 2: GND -> Net-(D10-A)
- J2 pad 1: Net-(J2-Pad1) -> Y+
- J3 pad 1: Net-(J3-Pad1) -> X+
- J4 pad 1: Net-(J4-Pad1) -> +15V
- J5 pad 1: Net-(J5-Pad1) -> Net-(J5-Pin_1)
- J6 pad 1: Net-(J6-Pad1) -> Net-(J6-Pin_1)
- J7 pad 1: Net-(J7-Pad1) -> Net-(J7-Pin_1)
- J8 pad 1: Net-(J8-Pad1) -> Net-(J8-Pin_1)
- J8 pad 5: Net-(J8-Pad5) -> Net-(J8-Pin_5)
- J9 pad 1: +15V -> Net-(D14-A)
- J9 pad 2: Net-(J11-Pad1) -> Net-(U6-VIN-)
- J9 pad 3: MOTOR_ON -> Net-(U6-VIN-)
- Q1 pad 1: Net-(Q1-Pad1) -> Net-(Q1-B)
- Q1 pad 2: Net-(J5-Pad1) -> Net-(J6-Pin_1)
- Q1 pad 3: Net-(Q1-Pad3) -> Net-(Q1-E)
- Q2 pad 1: Net-(Q2-Pad1) -> Net-(Q2-B)
- Q2 pad 2: Net-(J6-Pad1) -> Net-(J7-Pin_1)
- Q2 pad 3: Net-(Q2-Pad3) -> Net-(Q2-E)
- Q3 pad 1: Net-(Q3-Pad1) -> Net-(Q3-G)
- Q3 pad 2: Net-(J7-Pad1) -> GND
- Q3 pad 3: Net-(Q3-Pad3) -> Net-(D10-A)
- R10 pad 2: Net-(Q3-Pad3) -> Net-(Q2-B)
- R11 pad 1: Net-(Q2-Pad1) -> Net-(Q1-E)
- R12 pad 1: Net-(Q2-Pad1) -> Net-(Q1-E)
- R13 pad 1: Net-(Q2-Pad1) -> Net-(Q1-E)
- R14 pad 1: Net-(Q3-Pad1) -> Net-(Q2-E)
- R14 pad 2: Net-(J8-Pad1) -> Net-(J8-Pin_5)
- R15 pad 1: Net-(Q3-Pad1) -> Net-(Q2-E)
- R15 pad 2: Net-(J8-Pad1) -> Net-(J8-Pin_5)
- R16 pad 1: Net-(Q3-Pad1) -> Net-(Q2-E)
- R16 pad 2: Net-(J8-Pad1) -> Net-(J8-Pin_5)
- R17 pad 1: Net-(Q1-Pad1) -> Net-(Q4-E)
- R17 pad 2: Net-(J8-Pad5) -> Net-(J8-Pin_1)
- R18 pad 1: Net-(Q1-Pad1) -> Net-(Q4-E)
- R18 pad 2: Net-(J8-Pad5) -> Net-(J8-Pin_1)
- R19 pad 1: Net-(Q1-Pad1) -> Net-(Q4-E)
- R19 pad 2: Net-(J8-Pad5) -> Net-(J8-Pin_1)
- R20 pad 1: Net-(J8-Pad5) -> Net-(J8-Pin_1)
- R22 pad 1: Net-(J8-Pad1) -> Net-(J8-Pin_5)
- R27 pad 2: Net-(C15-Pad1) -> Net-(U3D-+)
- R5 pad 2: Net-(J2-Pad1) -> RED
- R6 pad 2: Net-(J3-Pad1) -> GREEN
- R7 pad 2: Net-(J4-Pad1) -> BLUE
- R8 pad 2: Net-(Q1-Pad3) -> Net-(Q4-B)
- R9 pad 2: Net-(Q2-Pad3) -> Net-(Q1-B)
- U2 pad 13: Net-(Q3-Pad1) -> Net-(Q2-E)
- U2 pad 2: Net-(Q2-Pad1) -> Net-(Q1-E)
- U2 pad 6: Net-(Q1-Pad1) -> Net-(Q4-E)
- U3 pad 12: Net-(C15-Pad1) -> Net-(U3D-+)
Routing:
- net Net-(Q4-E): track 0.00 -> 164.1 mm, vias 0 -> 1
- net BLUE: track 0.00 -> 150.4 mm, vias 0 -> 1
- net Net-(Q4-B): track 0.00 -> 146.2 mm, vias 0 -> 1
- net Net-(U2B-+): track 11.4 -> 147.4 mm, vias 0 -> 1
- net +12V: track 0.00 -> 134.5 mm, vias 0 -> 2
- net Net-(Q1-E): track 0.00 -> 134.2 mm, vias 0 -> 1
- net VCC: track 0.00 -> 131.3 mm, vias 0 -> 5
- net GREEN: track 0.00 -> 119.4 mm, vias 0 -> 1
- net +15V: track 12.8 -> 128.9 mm
- net Net-(Q1-B): track 0.00 -> 114.7 mm, vias 0 -> 1
- net Net-(U2A-+): track 10.2 -> 120.4 mm, vias 0 -> 1
- net Net-(Q2-E): track 0.00 -> 105.9 mm, vias 0 -> 1
- net Net-(J8-Pin_1): track 0.00 -> 103.8 mm
- net RED: track 0.00 -> 87.2 mm, vias 0 -> 1
- net -15V: track 0.00 -> 86.9 mm, vias 0 -> 2
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Other:
- board text added: "-15V G +15V"
- board text added: "15V"
- board text added: "AUTO OFF ENABLE"
- board text added: "BLUE - +"
- board text added: "GREEN - +"
- board text added: "RED - +"
- board text added: "X- G X+"
- board text added: "Y- G Y+"
- board text removed: "- TTL + BLUE"
- board text removed: "- TTL + GREEN"
- board text removed: "- TTL + RED"
- board text removed: "3.3V"
- board text removed: "7.5V"
- board text removed: "B- B+"
- board text removed: "G- G+"
- board text removed: "GND 12V"
- board text removed: "R- R+"
