File: hardware/mega_laser_driver/mega_laser_driver.kicad_sch (KiCad schematic)
At the start: 90 parts, among them J1 Conn_01x03, J10 Conn_01x02, J11 Conn_01x02, J2 Conn_01x02, J3 Conn_01x02, J4 Conn_01x02, J5 Conn_01x02, J6 Conn_01x02, J7 Conn_01x02, J8 Conn_02x03_Odd_Even, J9 Conn_01x03, K1 G6S-2, Q1 BD139, Q2 BD139, Q3 BD139, U1 LM2576S-ADJ, U2 LM324, U3 LM324, U4 LM2576S-ADJ, U5 LM2576S-ADJ

Commit message: Added new hardware
Parts:
- removed C15: 47u, Capacitor_SMD:CP_Elec_6.3x5.4_Nichicon, symbol Device:C_Polarized_US
- removed J1: Conn_01x03, Connector_JST:JST_XH_B3B-XH-A_1x03_P2.50mm_Vertical, symbol Connector_Generic:Conn_01x03
- removed J10, J2, J3, J4: Conn_01x02, Connector_JST:JST_XH_B2B-XH-A_1x02_P2.50mm_Vertical, symbol Connector_Generic:Conn_01x02
- removed J11: Conn_01x02, Connector_PinHeader_2.54mm:PinHeader_1x02_P2.54mm_Vertical, symbol Connector_Generic:Conn_01x02
- removed J9: Conn_01x03, Connector_PinHeader_2.54mm:PinHeader_1x03_P2.54mm_Vertical, symbol Connector_Generic:Conn_01x03
- removed K1: G6S-2, Relay_THT:Relay_DPDT_Omron_G6S-2, symbol Relay:G6S-2
- removed Q1, Q2, Q3: BD139, Package_TO_SOT_THT:TO-126-3_Horizontal_TabDown, symbol Transistor_BJT:BD139
- added C10, C11, C9: 220u, Capacitor_SMD:CP_Elec_6.3x7.7, symbol Device:C_Polarized_US
- added C15: 47u, Capacitor_SMD:C_1210_3225Metric, symbol Device:C
- added D1 (x2): LED, LED_SMD:LED_0603_1608Metric, symbol Device:LED
- added D4: SS54, Diode_SMD:D_SMA, symbol Diode:B320
- added J12: DB25_Plug_MountingHoles, Connector_Dsub:DSUB-25_Male_Horizontal_P2.77x2.84mm_EdgePinOffset7.70mm_Housed_MountingHolesOffset9.12mm, symbol Connector:DB25_Plug_MountingHoles
- added J2, J3, J4: Conn_01x03, Connector_JST:JST_XH_B3B-XH-A_1x03_P2.50mm_Vertical, symbol Connector_Generic:Conn_01x03
- added J2: Barrel_Jack_Switch, Connector_BarrelJack:BarrelJack_CLIFF_FC681465S_SMT_Horizontal, symbol Connector:Barrel_Jack_Switch
- added K2: G5Q-1A-DC12, Relay_THT:Relay_SPST_Omron-G5Q-1A, symbol Relay:G5Q-1A
- added Q1, Q2, Q4: TIP120, Package_TO_SOT_THT:TO-220-3_Horizontal_TabDown, symbol Transistor_BJT:TIP120
- added Q3: 2N7002, Package_TO_SOT_SMD:SOT-23, symbol Transistor_FET:2N7002
- added R24: 680, Resistor_SMD:R_0603_1608Metric, symbol Device:R
- added R24: 560, Resistor_SMD:R_0603_1608Metric, symbol Device:R
- added R31: 100, Resistor_SMD:R_0603_1608Metric, symbol Device:R_US
- added SW1: SW_SPDT, Button_Switch_SMD:SW_SPDT_PCM12, symbol Switch:SW_SPDT
- added U6: TEN20-2422WIN, AlexCustom:PYBE30-Q24-D15, symbol Converter_DCDC:TEN20-2422WIN
- C12, C13, C3, C4, C5, C6: value 1000u -> 220u; footprint Capacitor_SMD:CP_Elec_10x10 -> Capacitor_SMD:CP_Elec_6.3x7.7
- D1, D2, D9: footprint Diode_SMD:D_SMA_Handsoldering -> Diode_SMD:D_SOD-123
Connections:
- net +15V: now also C10.1, D1.2 (A), J4.1 (Pin_1), K2.3, U6.6 (VOUT+)
- net -15V: now also C11.2, J4.3 (Pin_3), U6.4 (VOUT-)
- net GND: now also C10.2, C11.1, C15.1, J12.0 (PAD), J12.18 (P18), J12.19 (P19), J12.20 (P20), J12.21 (P21), J12.22 (P22), J12.23 (P23), J12.25 (P25), J2.2 (Pin_2), J3.2 (Pin_2), J4.2 (Pin_2), Q3.2 (S), R24.2, R24.2, U6.5 (CM); no longer D10.2 (A)
- net MOTOR_ON: now also SW1.3 (C)
- net VCC: now also K2.2
- net RED: now reaches R5.2
- net RED: now also J12.5
- net BLUE: now reaches R7.2
- net BLUE: now also J12.7
- net at R11.1, R12.1, R13.1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: now also Q1.3 (E)
- net at J6.1 (Pin_1): now also Q1.2 (C)
- net at R9.2: now also Q1.1 (B)
- net X+: now reaches C14.1
- net X+: now also J12.1, J3.1 (Pin_1)
- net at R17.1, R18.1, R19.1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: now also Q4.3 (E)
- net at R17.2, R18.2, R19.2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: now also J8.1 (Pin_1); no longer J8.5 (Pin_5)
- net at R27.2, U3.12 (+): now also C15.2
- net GREEN: now reaches R6.2
- net GREEN: now also J12.6
- net +12V: now reaches D10.1 (K)
- net +12V: now also C9.1, D1.2 (A), D4.1 (K), K2.5, SW1.1 (A), U6.1 (VIN+)
- net at J5.1 (Pin_1): now also Q4.2 (C)
- net at R14.1, R15.1, R16.1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: now also Q2.3 (E)
- net at J7.1 (Pin_1): now also Q2.2 (C)
- net at R10.2: now also Q2.1 (B)
- net at R8.2: now also Q4.1 (B)
- net at R14.2, R15.2, R16.2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: now also J8.5 (Pin_5); no longer J8.1 (Pin_1)
- new net: D10.2 (A), K2.1, Q3.3 (D)
- new net: Q3.1 (G), R31.2
- new net: D1.1 (K), R24.1 (x2)
- new net: C9.2, J2.2, J2.3, U6.2 (VIN-)
- new net: D4.2 (A), J2.1
- new net INTERLOCK1: J12.4, R31.1
- new net INTERLOCK2: J12.17 (P17), SW1.2 (B)
- new net X-: J12.14 (P14), J3.3 (Pin_3)
- new net Y+: J12.2, J2.1 (Pin_1)
- new net Y-: J12.15 (P15), J2.3 (Pin_3)
Other:
- moved on the sheet: C1, C14, C2, C7, C8, D1, D10, D11, D12, D2, D9, H1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
